File: Hardware/Glasses Arms PCBs/Version 3.0/ESP32S3comV3.kicad_pcb (KiCad board)
At the start: 2 copper layers, 179.3 x 66.1 mm, 66 parts, among them J1 USB_C_Receptacle_USB2.0_16P, J2 USB_C_Receptacle_USB2.0_16P, J3 Connector_Generic:Conn_02x05_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, J4 Connector_Generic:Conn_02x05_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, J5 SFM-105-01-L-S, J6 SFM-105-01-L-S, J7 Conn_01x06, J8 Conn_01x06, J9 Conn_02x01, SW1 SW_Push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

Commit message: Update ESP32S3comV3.kicad_pcb
Routing:
- net GND: track 110.5 -> 111.1 mm, vias 46 -> 44
