File: Hardware/Glasses Arms PCBs/Version 3.1/ESP32R.kicad_sch (KiCad schematic)
At the start: 23 parts, among them J10 Conn_01x02, J11 Conn_01x08_Socket, J2 USB_C_Receptacle_USB2.0_16P, J3 Connector_Generic:Conn_02x05_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, Q1 BSS138, U2 LT1963AxST-3.3

Commit message: update
Parts:
- added SW2: OS102011MA1QN1, OS102011MA1QN1_CNK, symbol 2025-01-30_01-45-57:OS102011MA1QN1
Connections:
- net Bat: now also SW2.3
- net EN: now also SW2.2
- net GND: now also SW2.1
Changed lines of the file:
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@@
 	(wire
 		(pts
+			(xy 209.55 101.6) (xy 215.9 101.6)
+		)
+		(stroke
+			(width 0)
+			(type default)
+		)
+	)
+	(wire
+		(pts
 			(xy 107.95 179.07) (xy 120.65 179.07)
 		)
@@
 	(wire
 		(pts
+			(xy 209.55 99.06) (xy 212.09 99.06)
+		)
+		(stroke
+			(width 0)
+			(type default)
+		)
+	)
+	(wire
+		(pts
 			(xy 38.1 149.86) (xy 54.61 149.86)
 		)
@@
 	(wire
 		(pts
+			(xy 184.15 99.06) (xy 189.23 99.06)
+		)
+		(stroke
+			(width 0)
+			(type default)
+		)
+	)
+	(wire
+		(pts
 			(xy 128.27 73.66) (xy 149.86 73.66)
 		)
@@
 		)
 	)
+	(label "Bat"
+		(at 212.09 99.06 0)
+		(fields_autoplaced yes)
+		(effects
+			(font
+				(size 1.27 1.27)
+			)
+			(justify left bottom)
+		)
+	)
 	(label "GPIO11"
 		(at 120.65 179.07 0)
@@
 	)
 	(label "GND"
-		(at 129.54 55.88 0)
+		(at 184.15 99.06 0)
 		(fields_autoplaced yes)
 		(effects
@@
 	)
 	(label "EN"
-		(at 129.54 53.34 0)
+		(at 215.9 101.6 180)
 		(fields_autoplaced yes)
 		(effects
@@
 				(size 1.27 1.27)
 			)
-			(justify left bottom)
+			(justify right bottom)
 		)
 	)
@@
 					(unit 1)
 				)
+			)
+		)
+	)
+	(symbol
+		(lib_id "2025-01-30_01-45-57:OS102011MA1QN1")
+		(at 189.23 99.06 0)
+		(unit 1)
+		(exclude_from_sim no)
+		(in_bom yes)
+		(on_board yes)
+		(dnp no)
+		(fields_autoplaced yes)
+		(property "Reference" "SW2"
+			(at 199.39 91.44 0)
+			(effects
+				(font
+					(size 1.524 1.524)
+				)
+			)
+		)
+		(property "Value" "OS102011MA1QN1"
+			(at 199.39 93.98 0)
+			(effects
+				(font
+					(size 1.524 1.524)
+				)
+			)
+		)
+		(property "Footprint" "OS102011MA1QN1_CNK"
+			(at 189.23 99.06 0)
+			(effects
+				(font
+					(size 1.27 1.27)
+					(italic yes)
+				)
+				(hide yes)
+			)
+		)
+		(property "Datasheet" "OS102011MA1QN1"
+			(at 189.23 99.06 0)
+			(effects
+				(font
+					(size 1.27 1.27)
+					(italic yes)
+				)
+				(hide yes)
+			)
+		)
+		(property "Description" ""
+			(at 189.23 99.06 0)
+			(effects
+				(font
+					(size 1.27 1.27)
+				)
+				(hide yes)
+			)
+		)
+		(pin "3"
+		)
+		(pin "1"
+		)
+		(pin "2"
+		)
+		(instances
+			(project ""
+				(path "/d6aa16de-0937-4a13-9de5-3126c435d533/20542354-0dfe-41b3-9978-21e838dfcc86"
+					(reference "SW2")
+					(unit 1)
+				)
