File: Hardware/Glasses Arms PCBs/Version 3.1/ESP32S3comV3.1.kicad_pcb (KiCad board)
At the start: 2 copper layers, 179.3 x 66.1 mm, 66 parts, among them J1 USB_C_Receptacle_USB2.0_16P, J10 Conn_01x02, J11 Conn_01x08_Socket, J2 USB_C_Receptacle_USB2.0_16P, J3 Connector_Generic:Conn_02x05_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, J4 Connector_Generic:Conn_02x05_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, J5 BD050-10-A-0-0500-L-D, J6 BD050-10-A-0-0500-L-D, J7 Conn_02x06, J8 Conn_02x06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

Commit message: update
Parts:
- added SW2: OS102011MA1QN1, footprints:OS102011MA1QN1_CNK, F.Cu at (189.5, 92.2)
- moved R4 0.20 mm to (204.9, 120.3)
- moved MK5 0.15 mm to (208.1, 120.2)
Connections:
- J4 pad 1: /WS1 -> /GPIO13
- J4 pad 3: /SCK1 -> /GPIO14
- J4 pad 5: /SD1 -> /GPIO21
- J7 pad 8: unconnected-(J7-Pin_8-Pad8) -> /Eye connect/LB
- J8 pad 6: unconnected-(J8-Pin_6-Pad6) -> /Eye connect/LB
Routing:
- net /GPIO13: track 0.00 -> 34.8 mm, vias 0 -> 2
- net /GPIO14: track 0.00 -> 32.2 mm, vias 0 -> 2
- net /GPIO21: track 0.00 -> 29.9 mm, vias 0 -> 2
- net /BoardR/EN: track 0.00 -> 28.7 mm, vias 0 -> 1
- net /Eye connect/LB: track 0.00 -> 22.1 mm
- net /BoardR/Bat: track 14.9 -> 34.6 mm
- net GND: track 101.4 -> 111.2 mm, vias 38 -> 36
- net /GPIO2: track 165.5 -> 163.4 mm
- net /VCC_3V3: track 206.9 -> 208.7 mm
- net /BoardR/5V: track 39.4 -> 40.2 mm
- net /BoardR/VCC_3V3: track 199.5 -> 200.0 mm
