File: Hardware/Glasses Arms PCBs/Version 3.1/ESP32S3comV3.1.kicad_sch (KiCad schematic)
At the start: 29 parts, among them J1 USB_C_Receptacle_USB2.0_16P, J4 Connector_Generic:Conn_02x05_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, J9 Conn_02x01, SW1 SW_Push, U1 ESP32-S3-WROOM-1U-N8R8, U3 LT1963AxST-3.3

Commit message: update
Connections:
- net SCK1 is gone; now on net GPIO14: J4.3 (Pin_3)
- net SD1 is gone; now on net GPIO21: J4.5 (Pin_5)
- net WS1 is gone; now on net GPIO13: J4.1 (Pin_1)
- no-connect marks 23 -> 21
Changed lines of the file:
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@@
-	)
-	(no_connect
-		(at 120.65 83.82)
 	)
 	(no_connect
@@
 	)
 	(no_connect
-		(at 179.07 58.42)
-	)
-	(no_connect
 		(at 120.65 60.96)
 	)
@@
 	)
 	(no_connect
-		(at 120.65 81.28)
-	)
-	(no_connect
 		(at 54.61 60.96)
 	)
@@
 	)
 	(no_connect
+		(at 120.65 88.9)
+	)
+	(no_connect
 		(at 120.65 66.04)
 	)
@@
 	(wire
 		(pts
-			(xy 107.95 173.99) (xy 120.65 173.99)
+			(xy 110.49 166.37) (xy 123.19 166.37)
 		)
 		(stroke
@@
 	(wire
 		(pts
-			(xy 107.95 179.07) (xy 120.65 179.07)
+			(xy 110.49 171.45) (xy 123.19 171.45)
 		)
 		(stroke
@@
 	(wire
 		(pts
-			(xy 107.95 181.61) (xy 120.65 181.61)
+			(xy 110.49 173.99) (xy 123.19 173.99)
 		)
 		(stroke
@@
 	(wire
 		(pts
-			(xy 107.95 176.53) (xy 120.65 176.53)
+			(xy 110.49 168.91) (xy 123.19 168.91)
 		)
 		(stroke
@@
 	(text "SPI\n"
 		(exclude_from_sim no)
-		(at 131.318 176.784 0)
+		(at 133.858 169.164 0)
 		(effects
 			(font
@@
 	)
 	(label "GPIO12"
-		(at 120.65 181.61 0)
+		(at 123.19 173.99 0)
 		(fields_autoplaced yes)
 		(effects
@@
 	)
 	(label "MISO"
-		(at 107.95 176.53 0)
+		(at 110.49 168.91 0)
 		(fields_autoplaced yes)
 		(effects
@@
 	)
 	(label "MOSI"
-		(at 107.95 173.99 0)
+		(at 110.49 166.37 0)
 		(fields_autoplaced yes)
 		(effects
@@
 	)
 	(label "GPIO11"
-		(at 120.65 179.07 0)
+		(at 123.19 171.45 0)
 		(fields_autoplaced yes)
 		(effects
@@
 		)
 	)
+	(label "GPIO14"
+		(at 129.54 160.02 180)
+		(fields_autoplaced yes)
+		(effects
+			(font
+				(size 1.27 1.27)
+			)
+			(justify right bottom)
+		)
+	)
 	(label "GPIO16"
 		(at 120.65 88.9 0)
@@
 	)
 	(label "SCLK"
-		(at 107.95 179.07 0)
+		(at 110.49 171.45 0)
 		(fields_autoplaced yes)
 		(effects
@@
 	)
 	(label "GPIO10"
-		(at 120.65 176.53 0)
-		(fields_autoplaced yes)
-		(effects
-			(font
-				(size 1.27 1.27)
-			)
-			(justify left bottom)
+		(at 123.19 168.91 0)
+		(fields_autoplaced yes)
+		(effects
+			(font
+				(size 1.27 1.27)
+			)
+			(justify left bottom)
+		)
+	)
+	(label "GPIO13"
+		(at 129.54 157.48 180)
+		(fields_autoplaced yes)
+		(effects
+			(font
+				(size 1.27 1.27)
+			)
+			(justify right bottom)
 		)
 	)
@@
 	)
 	(label "GPIO21"
+		(at 129.54 162.56 180)
+		(fields_autoplaced yes)
+		(effects
+			(font
+				(size 1.27 1.27)
+			)
+			(justify right bottom)
+		)
+	)
+	(label "GPIO21"
 		(at 179.07 58.42 180)
 		(fields_autoplaced yes)
@@
 	)
 	(label "SC"
-		(at 107.95 181.61 0)
+		(at 110.49 173.99 0)
 		(fields_autoplaced yes)
 		(effects
@@
 	)
 	(label "GPIO9"
-		(at 120.65 173.99 0)
-		(fields_autoplaced yes)
-		(effects
+		(at 123.19 166.37 0)
+		(fields_autoplaced yes)
+		(effects
