File: Hardware/Glasses Arms PCBs/Version 3.1/esp32s3eye breakout.kicad_sch (KiCad schematic)
At the start: 6 parts, among them J1 BD050-10-A-0-0500-L-D, J2 BD050-10-A-0-0500-L-D, J7 Conn_02x06, J8 Conn_02x06

Commit message: update
Connections:
- net LB: now reaches J7.8 (Pin_8)
- net LB: now also J8.6 (Pin_6)
Changed lines of the file:
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@@
+	(wire
+		(pts
+			(xy 175.26 97.79) (xy 186.69 97.79)
+		)
+		(stroke
+			(width 0)
+			(type default)
+		)
+	)
 	(wire
 		(pts
@@
 	(wire
 		(pts
+			(xy 218.44 123.19) (xy 228.6 123.19)
+		)
+		(stroke
+			(width 0)
+			(type default)
+		)
+	)
+	(wire
+		(pts
 			(xy 199.39 92.71) (xy 209.55 92.71)
 		)
@@
 			(width 0)
 			(type default)
+		)
+	)
+	(label "LB"
+		(at 228.6 123.19 180)
+		(fields_autoplaced yes)
+		(effects
+			(font
+				(size 1.27 1.27)
+			)
+			(justify right bottom)
 		)
 	)
@@
 		(fields_autoplaced yes)
 		(effects
+			(font
+				(size 1.27 1.27)
+			)
+			(justify left bottom)
+		)
+	)
+	(label "LB"
+		(at 175.26 97.79 0)
+		(fields_autoplaced yes)
+		(effects
