File: Hardware/Glasses Arms PCBs/Version 3.3/ESP32S3comV3.3.kicad_pcb (KiCad board)
At the start: 2 copper layers, 179.3 x 66.1 mm, 66 parts, among them J1 USB_C_Receptacle_USB2.0_16P, J2 USB_C_Receptacle_USB2.0_16P, J3 Connector_Generic:Conn_02x05_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, J4 Connector_Generic:Conn_02x05_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, J5 BD050-10-A-0-0500-L-D, J6 BD050-10-A-0-0500-L-D, J7 Conn_01x06, J8 Conn_01x06, J9 Conn_02x01, SW1 SW_Push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

Commit message: update
Other:
- board text added: "AR Glass V3.3 1/25"
- board text removed: "AR Glass V3 1/25"
- board text removed: "AR Glass V3.0 1/25"
Changed lines of the file:
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@@
 		)
 	)
-	(gr_text "AR Glass\nV3\n1/25\n"
+	(gr_text "AR Glass\nV3.3\n1/25\n"
 		(at 200.52 92.47 180)
 		(layer "F.SilkS")
@@
 		)
 	)
-	(gr_text "AR Glass\nV3.0\n1/25\n"
+	(gr_text "AR Glass\nV3.3\n1/25\n"
 		(at 159.847002 138.910776 0)
 		(layer "F.SilkS")
