File: Hardware/Glasses Arms PCBs/Version 3.2/ESP32S3comV3.2.kicad_pcb (KiCad board)
At the start: 2 copper layers, 179.3 x 66.1 mm, 69 parts, among them J1 USB_C_Receptacle_USB2.0_16P, J10 Conn_01x02, J11 Conn_01x08_Socket, J2 USB_C_Receptacle_USB2.0_16P, J3 PinSocket_2x05_P2.00mm_Vertic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, J4 PinSocket_2x05_P2.00mm_Vertic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, J5 BD050-10-A-0-0500-L-D, J6 BD050-10-A-0-0500-L-D, J7 PinHeader_2x06_P2.54mm_Vertic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, J8 PinHeader_2x06_P2.54mm_Vertic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

Commit message: update
Other:
- board text added: "AR Glass V3.2 1/25"
- board text removed: "AR Glass V3.1 1/25"
Changed lines of the file:
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@@
 		)
 	)
-	(gr_text "AR Glass\nV3.1\n1/25\n"
+	(gr_text "AR Glass\nV3.2\n1/25\n"
 		(at 200.52 92.47 180)
 		(layer "F.SilkS")
@@
 		)
 	)
-	(gr_text "AR Glass\nV3.1\n1/25\n"
+	(gr_text "AR Glass\nV3.2\n1/25\n"
 		(at 159.847002 138.910776 0)
 		(layer "F.SilkS")

Commit message: update
Routing:
- net /GPIO2: track 149.3 -> 147.9 mm, vias 3 -> 2
Changed lines of the file:
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@@
+	)
+	(segment
+		(start 202.525 122.525)
+		(end 202.52 122.52)
+		(width 0.2)
+		(layer "F.Cu")
+		(net 23)
+	)
+	(segment
+		(start 202.52 122.52)
+		(end 188.93 122.52)
+		(width 0.2)
+		(layer "F.Cu")
+		(net 23)
 	)
 	(segment
@@
 	)
 	(segment
-		(start 76.9763 137.8652)
-		(end 75.6373 137.8652)
+		(start 186.35 123.75)
+		(end 187.58 122.52)
 		(width 0.2)
 		(layer "F.Cu")
@@
 	)
 	(segment
-		(start 190.22 122.52)
-		(end 188.93 122.52)
+		(start 76.9763 137.8652)
+		(end 75.6373 137.8652)
 		(width 0.2)
 		(layer "F.Cu")
@@
 	)
 	(segment
-		(start 191.275 123.575)
-		(end 190.22 122.52)
+		(start 187.58 122.52)
+		(end 188.93 122.52)
 		(width 0.2)
 		(layer "F.Cu")
@@
 	)
 	(via
-		(at 191.275 123.575)
+		(at 186.35 123.75)
 		(size 0.6)
 		(drill 0.3)
@@
 		(net 23)
 	)
-	(via
-		(at 202.525 122.525)
-		(size 0.6)
-		(drill 0.3)
-		(layers "F.Cu" "B.Cu")
-		(net 23)
-	)
 	(segment
-		(start 185.3 127.175)
-		(end 150.489215 127.175)
+		(start 148.964215 125.65)
+		(end 89.1915 125.65)
 		(width 0.2)
 		(layer "B.Cu")
@@
 	)
 	(segment
+		(start 186.35 126.125)
+		(end 185.3 127.175)
+		(width 0.2)
+		(layer "B.Cu")
+		(net 23)
+	)
+	(segment
 		(start 89.1915 125.65)
 		(end 76.9763 137.8652)
@@
 	)
 	(segment
-		(start 148.964215 125.65)
-		(end 89.1915 125.65)
+		(start 186.35 123.75)
+		(end 186.35 126.125)
 		(width 0.2)
 		(layer "B.Cu")
@@
 	)
 	(segment
-		(start 188.9 123.575)
-		(end 185.3 127.175)
+		(start 185.3 127.175)
+		(end 150.489215 127.175)
 		(width 0.2)
 		(layer "B.Cu")
-		(net 23)
-	)
-	(segment
-		(start 201.475 123.575)
-		(end 191.275 123.575)
-		(width 0.2)
-		(layer "B.Cu")
-		(net 23)
-	)
-	(segment
-		(start 202.525 122.525)
-		(end 201.475 123.575)
-		(width 0.2)
-		(layer "B.Cu")
-		(net 23)
-	)
-	(segment
-		(start 191.275 123.575)
-		(end 188.9 123.575)
-		(width 0.2)
-		(layer "B.Cu")

Commit message: update
Parts:
- moved H1 1.04 mm to (219.1, 104.5)
- moved H2 1.03 mm to (242.0, 104.5)
- moved H4 0.11 mm to (219.1, 128.4)
Changed lines of the file:
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@@
 		(tags "Through hole pin header THT 2x06 2.54mm double row")
 		(property "Reference" "J8"
-			(at -0.05 -3.105 180)
+			(at 5.525 -0.08 180)
 			(layer "F.SilkS")
 			(effects
@@
 	(footprint "MountingHole:MountingHole_2.2mm_M2_DIN965_Pad"
 		(layer "F.Cu")
-		(at 219 128.275)
+		(at 219.05 128.375)
 		(descr "Mounting Hole 2.2mm, M2, DIN965")
 		(tags "mounting hole 2.2mm m2 din965")
@@
 	(footprint "MountingHole:MountingHole_2.2mm_M2_DIN965_Pad"
 		(layer "F.Cu")
-		(at 218.85 105.525)
+		(at 219.05 104.5)
 		(descr "Mounting Hole 2.2mm, M2, DIN965")
 		(tags "mounting hole 2.2mm m2 din965")
 		(property "Reference" "H1"
-			(at 0 -2.9 0)
+			(at 0.025 3.025 0)
 			(layer "F.SilkS")
 			(effects
@@
 	(footprint "MountingHole:MountingHole_2.2mm_M2_DIN965_Pad"
 		(layer "F.Cu")
-		(at 241.31 103.735)
+		(at 242 104.5)
 		(descr "Mounting Hole 2.2mm, M2, DIN965")
 		(tags "mounting hole 2.2mm m2 din965")
 		(property "Reference" "H2"
-			(at -0.285 3.415 0)
+			(at -0.025 3.25 0)
 			(layer "F.SilkS")
 			(effects

Commit message: update
Parts:
- moved J8 0.92 mm to (224.3, 110.0)
Connections:
- J7 pad 10: unconnected-(J7-Pin_10-Pad10) -> /Eye connect/LB
- J7 pad 2: /Eye connect/WS1 -> /Eye connect/VCC_3V3
- J7 pad 4: /Eye connect/SCK1 -> /Eye connect/WS1
- J7 pad 6: /Eye connect/SD1 -> /Eye connect/SCK1
- J7 pad 8: /Eye connect/LB -> /Eye connect/SD1
Routing:
- net /Eye connect/VCC_3V3: track 7.17 -> 24.9 mm
- net /Eye connect/LB: track 22.1 -> 22.8 mm
- net /Eye connect/SD1: track 22.1 -> 22.7 mm
- net GND: track 115.0 -> 115.6 mm
- net /Eye connect/SCK1: track 22.1 -> 22.7 mm
- net /Eye connect/WS1: track 22.1 -> 22.7 mm
Other:
- board text added: "5V Gn LB Gd EN Bat Gn IN"
- board text added: "AR Glass V3.2 2/25"
- board text added: "Gnd WS 3V3 Sck x SDout x SDin x LB"
- board text added: "LB SD SCK WS"
- board text added: "LB SD SCK WS 3v3"
- board text removed: "AR Glass V3.2 1/25"

Commit message: update
Routing:
- net /BoardR/SDin: track 169.8 -> 170.4 mm
- net /BoardR/WS: track 150.3 -> 150.8 mm
