File: Hardware/Glasses Arms PCBs/Version 3.2/ESP32R.kicad_sch (KiCad schematic)
At the start: 24 parts, among them J10 Conn_01x02, J11 Conn_01x08_Socket, J2 USB_C_Receptacle_USB2.0_16P, J3 PinSocket_2x05_P2.00mm_Vertic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, Q1 BSS138, SW2 OS102011MA1QN1, U2 LT1963AxST-3.3

Commit message: update
Other:
- note added: "Microphone and board-to-board connections"
Changed lines of the file:
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@@
+		)
+	)
+	(text "Microphone and board-to-board connections\n"
+		(exclude_from_sim no)
+		(at 46.228 187.452 0)
+		(effects
+			(font
+				(size 1.27 1.27)
+			)
 		)
 	)

Commit message: update
Connections:
- net LB3v3 is gone; now on net LB: J3.2 (Pin_2), Q1.2 (S), R10.2
- net SCK renamed SCK1
- net SDin renamed SD1
- net WS renamed WS1
Other:
- note added: "Board to eye connector"
- note added: "Low Battery Indicator"
- note added: "USB for Charging"
- note added: "Voltage regulator"
- note removed: "SPI"
- note removed: "UART or I2C"
- company: (none) -> OSHE - IRL Sub-Titles
- moved on the sheet: C10, C11, C16, C18, C19, C20, D7, J10, J11, J3, MK3, MK4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
