File: Hardware/Glasses Arms PCBs/Version 3.2/ESP32S3comV3.2.kicad_sch (KiCad schematic)
At the start: 29 parts, among them J1 USB_C_Receptacle_USB2.0_16P, J4 PinSocket_2x05_P2.00mm_Vertic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, J9 Conn_02x01, SW1 SW_Push, U1 ESP32-S3-WROOM-1U-N8R8, U3 LT1963AEST-3.3

Commit message: update
Other:
- note added: "Board to board connector"
- note added: "Connetions"
- note added: "I2S Mics"
Changed lines of the file:
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@@
 	(wire
 		(pts
-			(xy 110.49 147.32) (xy 129.54 147.32)
+			(xy 118.11 147.32) (xy 137.16 147.32)
 		)
 		(stroke
@@
 	(wire
 		(pts
-			(xy 110.49 166.37) (xy 123.19 166.37)
+			(xy 118.11 166.37) (xy 130.81 166.37)
 		)
 		(stroke
@@
 	(wire
 		(pts
-			(xy 110.49 162.56) (xy 129.54 162.56)
+			(xy 118.11 162.56) (xy 137.16 162.56)
 		)
 		(stroke
@@
 	(wire
 		(pts
-			(xy 110.49 144.78) (xy 129.54 144.78)
+			(xy 118.11 144.78) (xy 137.16 144.78)
 		)
 		(stroke
@@
 	(wire
 		(pts
-			(xy 110.49 160.02) (xy 129.54 160.02)
+			(xy 118.11 160.02) (xy 137.16 160.02)
 		)
 		(stroke
@@
 	(wire
 		(pts
-			(xy 110.49 171.45) (xy 123.19 171.45)
+			(xy 118.11 171.45) (xy 130.81 171.45)
 		)
 		(stroke
@@
 	(wire
 		(pts
-			(xy 110.49 173.99) (xy 123.19 173.99)
+			(xy 118.11 173.99) (xy 130.81 173.99)
 		)
 		(stroke
@@
 	(wire
 		(pts
-			(xy 110.49 152.4) (xy 129.54 152.4)
+			(xy 118.11 152.4) (xy 137.16 152.4)
 		)
 		(stroke
@@
 	(wire
 		(pts
-			(xy 110.49 149.86) (xy 129.54 149.86)
+			(xy 118.11 149.86) (xy 137.16 149.86)
 		)
 		(stroke
@@
 	(wire
 		(pts
-			(xy 110.49 168.91) (xy 123.19 168.91)
+			(xy 118.11 168.91) (xy 130.81 168.91)
 		)
 		(stroke
@@
 	(wire
 		(pts
-			(xy 110.49 157.48) (xy 129.54 157.48)
+			(xy 118.11 157.48) (xy 137.16 157.48)
 		)
 		(stroke
@@
 	(rectangle
 		(start 19.05 110.49)
-		(end 143.51 191.77)
+		(end 97.79 171.45)
 		(stroke
 			(width 0)
@@
 		)
 	)
+	(rectangle
+		(start 99.06 109.22)
+		(end 142.24 139.7)
+		(stroke
+			(width 0)
+			(type default)
+		)
+		(fill
+			(type none)
+		)
+	)
+	(rectangle
+		(start 99.06 140.97)
+		(end 147.32 176.53)
+		(stroke
+			(width 0)
+			(type default)
+		)
+		(fill
+			(type none)
+		)
+	)
+	(text "Board to board connector"
+		(exclude_from_sim no)
+		(at 117.856 111.506 0)
+		(effects
+			(font
+				(size 1.27 1.27)
+			)
+		)
+	)
 	(text "I2S board 2"
 		(exclude_from_sim no)
-		(at 101.6 159.258 0)
+		(at 109.22 159.258 0)
 		(effects
 			(font
@@
 	(text "SPI\n"
 		(exclude_from_sim no)
-		(at 133.858 169.164 0)
+		(at 141.478 169.164 0)
+		(effects
+			(font
+				(size 1.27 1.27)
+			)
+		)
+	)
+	(text "I2S Mics "
+		(exclude_from_sim no)
+		(at 27.94 115.316 0)
 		(effects
 			(font
@@
 	(text "I2S"
 		(exclude_from_sim no)
-		(at 134.112 148.336 0)
+		(at 141.732 148.336 0)
+		(effects
+			(font
+				(size 1.27 1.27)
+			)
+		)
+	)
+	(text "Connetions\n\n"
+		(exclude_from_sim no)
+		(at 106.172 174.752 0)
 		(effects
 			(font
@@
 	)
 	(label "GPIO42"
-		(at 129.54 144.78 180)
+		(at 137.16 144.78 180)
 		(fields_autoplaced yes)
 		(effects
@@
 	)
 	(label "GPIO12"
-		(at 123.19 173.99 0)
+		(at 130.81 173.99 0)
 		(fields_autoplaced yes)
 		(effects
@@
 	)
 	(label "GPIO41"
-		(at 129.54 147.32 180)
+		(at 137.16 147.32 180)
 		(fields_autoplaced yes)
 		(effects
@@
 	)
 	(label "SCK"
-		(at 110.49 147.32 0)
+		(at 118.11 147.32 0)
 		(fields_autoplaced yes)
 		(effects
@@
 	)
 	(label "SD1"
-		(at 110.49 162.56 0)
+		(at 118.11 162.56 0)
 		(fields_autoplaced yes)
 		(effects
@@
 	)
 	(label "MISO"
-		(at 110.49 168.91 0)
+		(at 118.11 168.91 0)
 		(fields_autoplaced yes)
 		(effects
@@
 	)
 	(label "WS1"
-		(at 110.49 157.48 0)
+		(at 118.11 157.48 0)
 		(fields_autoplaced yes)
 		(effects
@@
 	)
 	(label "MOSI"
-		(at 110.49 166.37 0)
+		(at 118.11 166.37 0)
 		(fields_autoplaced yes)
 		(effects
@@
 	)
 	(label "GPIO11"
-		(at 123.19 171.45 0)
+		(at 130.81 171.45 0)
 		(fields_autoplaced yes)
 		(effects
@@
 	)
 	(label "WS"
-		(at 110.49 144.78 0)
+		(at 118.11 144.78 0)
 		(fields_autoplaced yes)
 		(effects
@@
 	)
 	(label "GPIO14"
-		(at 129.54 160.02 180)
+		(at 137.16 160.02 180)
 		(fields_autoplaced yes)
 		(effects
@@
 	)
 	(label "SCLK"
-		(at 110.49 171.45 0)
+		(at 118.11 171.45 0)
 		(fields_autoplaced yes)
 		(effects
@@
 	)
 	(label "SDin"
-		(at 110.49 152.4 0)
+		(at 118.11 152.4 0)
 		(fields_autoplaced yes)
 		(effects
@@
 	)
 	(label "GPIO2"
-		(at 129.54 152.4 180)
+		(at 137.16 152.4 180)
 		(fields_autoplaced yes)
 		(effects
@@
 	)
 	(label "GPIO10"
-		(at 123.19 168.91 0)
+		(at 130.81 168.91 0)
 		(fields_autoplaced yes)
 		(effects
@@
 	)
 	(label "GPIO13"
-		(at 129.54 157.48 180)
+		(at 137.16 157.48 180)
 		(fields_autoplaced yes)
 		(effects
@@
 	)
 	(label "GPIO21"
-		(at 129.54 162.56 180)
+		(at 137.16 162.56 180)
 		(fields_autoplaced yes)
 		(effects
@@
 	)
 	(label "SDout"
-		(at 110.49 149.86 0)
+		(at 118.11 149.86 0)
 		(fields_autoplaced yes)
 		(effects
@@
 	)
 	(label "SCK1"
-		(at 110.49 160.02 0)
+		(at 118.11 160.02 0)
 		(fields_autoplaced yes)
 		(effects
@@
 	)
 	(label "GPIO2"
-		(at 129.54 149.86 180)
+		(at 137.16 149.86 180)
 		(fields_autoplaced yes)
 		(effects
@@
 	)
 	(label "SC"
-		(at 110.49 173.99 0)
+		(at 118.11 173.99 0)
 		(fields_autoplaced yes)
 		(effects
@@
 	)
 	(label "GPIO9"
-		(at 123.19 166.37 0)
-		(fields_autoplaced yes)
-		(effects
+		(at 130.81 166.37 0)
+		(fields_autoplaced yes)
+		(effects

Commit message: update
Other:
- note added: "Board to eye adapter connector"
- note removed: "Board to board connector"
- moved on the sheet: J4, J9
Changed lines of the file:
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@@
 	(wire
 		(pts
-			(xy 115.57 120.65) (xy 105.41 120.65)
+			(xy 185.42 142.24) (xy 175.26 142.24)
 		)
 		(stroke
@@
 	(wire
 		(pts
-			(xy 137.16 128.27) (xy 128.27 128.27)
+			(xy 207.01 149.86) (xy 198.12 149.86)
 		)
 		(stroke
@@
 	(wire
 		(pts
-			(xy 128.27 123.19) (xy 137.16 123.19)
+			(xy 198.12 144.78) (xy 207.01 144.78)
 		)
 		(stroke
@@
 	(wire
 		(pts
-			(xy 175.26 154.94) (xy 181.61 154.94)
+			(xy 128.27 125.73) (xy 134.62 125.73)
 		)
 		(stroke
@@
 	(wire
 		(pts
-			(xy 105.41 128.27) (xy 115.57 128.27)
+			(xy 175.26 149.86) (xy 185.42 149.86)
 		)
 		(stroke
@@
 	(wire
 		(pts
-			(xy 157.48 154.94) (xy 162.56 154.94)
+			(xy 110.49 125.73) (xy 115.57 125.73)
 		)
 		(stroke
@@
 	(wire
 		(pts
-			(xy 106.68 130.81) (xy 106.68 132.08)
+			(xy 176.53 152.4) (xy 176.53 153.67)
 		)
 		(stroke
@@
 	(wire
 		(pts
-			(xy 105.41 125.73) (xy 115.57 125.73)
+			(xy 175.26 147.32) (xy 185.42 147.32)
 		)
 		(stroke
@@
 	(wire
 		(pts
-			(xy 137.16 125.73) (xy 128.27 125.73)
+			(xy 207.01 147.32) (xy 198.12 147.32)
 		)
 		(stroke
@@
 	(wire
 		(pts
-			(xy 128.27 120.65) (xy 137.16 120.65)
+			(xy 198.12 142.24) (xy 207.01 142.24)
 		)
 		(stroke
@@
 	(wire
 		(pts
-			(xy 115.57 130.81) (xy 106.68 130.81)
+			(xy 185.42 152.4) (xy 176.53 152.4)
 		)
 		(stroke
@@
 	(wire
 		(pts
-			(xy 137.16 130.81) (xy 128.27 130.81)
+			(xy 207.01 152.4) (xy 198.12 152.4)
 		)
 		(stroke
@@
 	(wire
 		(pts
-			(xy 105.41 123.19) (xy 115.57 123.19)
+			(xy 175.26 144.78) (xy 185.42 144.78)
 		)
 		(stroke
@@
 	)
 	(rectangle
-		(start 99.06 109.22)
-		(end 142.24 139.7)
+		(start 168.91 130.81)
+		(end 212.09 161.29)
 		(stroke
 			(width 0)
@@
 		)
 	)
-	(text "Board to board connector"
+	(text "Board to eye adapter connector"
 		(exclude_from_sim no)
-		(at 117.856 111.506 0)
+		(at 187.706 133.096 0)
 		(effects
 			(font
@@
 	(text "I2S board 2"
 		(exclude_from_sim no)
-		(at 105.918 117.094 0)
+		(at 175.768 138.684 0)
 		(effects
 			(font
@@
 	(text "SPI out\n"
 		(exclude_from_sim no)
-		(at 132.842 133.604 0)
+		(at 202.692 155.194 0)
 		(effects
 			(font
@@
 	)
 	(label "VBUS"
-		(at 181.61 154.94 0)
+		(at 134.62 125.73 0)
 		(fields_autoplaced yes)
 		(effects
@@
 	)
 	(label "MOSI"
-		(at 137.16 123.19 180)
+		(at 207.01 144.78 180)
 		(fields_autoplaced yes)
 		(effects
@@
 	)
 	(label "SCLK"
-		(at 137.16 128.27 180)
+		(at 207.01 149.86 180)
 		(fields_autoplaced yes)
 		(effects
@@
 	)
 	(label "VCC_3V3"
-		(at 105.41 128.27 0)
+		(at 175.26 149.86 0)
 		(fields_autoplaced yes)
 		(effects
@@
 	)
 	(label "GPIO15"
-		(at 137.16 120.65 180)
+		(at 207.01 142.24 180)
 		(fields_autoplaced yes)
 		(effects
@@
 	)
 	(label "SCK1"
-		(at 105.41 123.19 0)
+		(at 175.26 144.78 0)
 		(fields_autoplaced yes)
 		(effects
@@
 	)
 	(label "WS1"
-		(at 105.41 120.65 0)
+		(at 175.26 142.24 0)
 		(fields_autoplaced yes)
 		(effects
@@
 	)
 	(label "SD1"
-		(at 105.41 125.73 0)
+		(at 175.26 147.32 0)
 		(fields_autoplaced yes)
 		(effects
@@
 	)
 	(label "SC"
-		(at 137.16 130.81 180)
+		(at 207.01 152.4 180)
 		(fields_autoplaced yes)
 		(effects
@@
 	)
 	(label "MISO"
-		(at 137.16 125.73 180)
+		(at 207.01 147.32 180)
 		(fields_autoplaced yes)
 		(effects
@@
 	(symbol
 		(lib_id "power:GND")
-		(at 157.48 154.94 0)
+		(at 110.49 125.73 0)
 		(unit 1)
 		(exclude_from_sim no)
@@
 		(fields_autoplaced yes)
 		(property "Reference" "#PWR018"
-			(at 157.48 161.29 0)
+			(at 110.49 132.08 0)
 			(effects
 				(font
@@
 		)
 		(property "Value" "GND"
-			(at 157.48 160.02 0)
+			(at 110.49 130.81 0)
 			(effects
 				(font
@@
 		)
 		(property "Footprint" ""
-			(at 157.48 154.94 0)
+			(at 110.49 125.73 0)
 			(effects
 				(font
@@
 		)
 		(property "Datasheet" ""
-			(at 157.48 154.94 0)
+			(at 110.49 125.73 0)
 			(effects
 				(font
@@
 		)
 		(property "Description" "Power symbol creates a global label with name \"GND\" , ground"
-			(at 157.48 154.94 0)
+			(at 110.49 125.73 0)
 			(effects
 				(font
@@
 	(symbol
 		(lib_id "Connector_Generic:Conn_02x05_Odd_Even")
-		(at 120.65 125.73 0)
+		(at 190.5 147.32 0)
 		(unit 1)
 		(exclude_from_sim no)
@@
 		(fields_autoplaced yes)
 		(property "Reference" "J4"
-			(at 121.92 116.84 0)
+			(at 191.77 138.43 0)
 			(effects
 				(font
@@
 		)
 		(property "Value" "PinSocket_2x05_P2.00mm_Vertical"
-			(at 121.92 119.38 0)
+			(at 191.77 140.97 0)
 			(effects
 				(font
@@
 		)
 		(property "Footprint" "Connector_PinSocket_2.00mm:PinSocket_2x05_P2.00mm_Vertical"
-			(at 120.65 125.73 0)
+			(at 190.5 147.32 0)
 			(effects
 				(font
@@
 		)
 		(property "Datasheet" "~"
-			(at 120.65 125.73 0)
+			(at 190.5 147.32 0)
 			(effects
 				(font
@@
 		)
 		(property "Description" "Generic connector, double row, 02x05, odd/even pin numbering scheme (row 1 odd numbers, row 2 even numbers), script generated (kicad-library-utils/schlib/autogen/connector/)"
-			(at 120.65 125.73 0)
+			(at 190.5 147.32 0)
 			(effects
 				(font
@@
 		)
 		(property "MANUFACTURER" ""
-			(at 120.65 125.73 0)
+			(at 190.5 147.32 0)
 			(effects
 				(font
@@
 		)
 		(property "MAXIMUM_PACKAGE_HEIGHT" ""
-			(at 120.65 125.73 0)
+			(at 190.5 147.32 0)
 			(effects
 				(font
@@
 		)
 		(property "PARTREV" ""
-			(at 120.65 125.73 0)
+			(at 190.5 147.32 0)
 			(effects
 				(font
@@
 		)
 		(property "SNAPEDA_PN" ""
-			(at 120.65 125.73 0)
+			(at 190.5 147.32 0)
 			(effects
 				(font
@@
 		)
 		(property "STANDARD" ""
-			(at 120.65 125.73 0)
+			(at 190.5 147.32 0)
 			(effects
 				(font
@@
 	(symbol
 		(lib_id "power:GND")
-		(at 106.68 132.08 0)
+		(at 176.53 153.67 0)
 		(unit 1)
 		(exclude_from_sim no)
@@
 		(fields_autoplaced yes)
 		(property "Reference" "#PWR03"
-			(at 106.68 138.43 0)
+			(at 176.53 160.02 0)
 			(effects
 				(font
@@
 		)
 		(property "Value" "GND"
-			(at 106.68 137.16 0)
+			(at 176.53 158.75 0)
 			(effects
 				(font
@@
 		)
 		(property "Footprint" ""
-			(at 106.68 132.08 0)
+			(at 176.53 153.67 0)
 			(effects
 				(font
@@
 		)
 		(property "Datasheet" ""
-			(at 106.68 132.08 0)
+			(at 176.53 153.67 0)
 			(effects
 				(font
@@
 		)
 		(property "Description" "Power symbol creates a global label with name \"GND\" , ground"
-			(at 106.68 132.08 0)
+			(at 176.53 153.67 0)
 			(effects
 				(font
@@
 	(symbol
 		(lib_id "Connector_Generic:Conn_02x01")
-		(at 170.18 154.94 180)
+		(at 123.19 125.73 180)
 		(unit 1)
 		(exclude_from_sim no)
@@
 		(fields_autoplaced yes)
 		(property "Reference" "J9"
-			(at 168.91 148.59 0)
+			(at 121.92 119.38 0)
 			(effects
 				(font
@@
 		)
 		(property "Value" "Conn_02x01"
-			(at 168.91 151.13 0)
+			(at 121.92 121.92 0)
 			(effects
 				(font
@@
 		)
 		(property "Footprint" "Connector_JST:JST_PH_B2B-PH-K_1x02_P2.00mm_Vertical"
-			(at 170.18 154.94 0)
+			(at 123.19 125.73 0)
 			(effects
 				(font
@@
 		)
 		(property "Datasheet" "~"
-			(at 170.18 154.94 0)
+			(at 123.19 125.73 0)
 			(effects
 				(font
@@
 		)
 		(property "Description" "Generic connector, double row, 02x01, this symbol is compatible with counter-clockwise, top-bottom and odd-even numbering schemes., script generated (kicad-library-utils/schlib/autogen/connector/)"
-			(at 170.18 154.94 0)
+			(at 123.19 125.73 0)
 			(effects
 				(font

Commit message: update
Parts:
- removed C1, C2: 0.1uF, Capacitor_SMD:C_0805_2012Metric_Pad1.18x1.45mm_HandSolder, symbol Device:C_Small
- removed C14, C4, C6, C7: 0.1uF, Capacitor_SMD:C_0805_2012Metric_Pad1.18x1.45mm_HandSolder, symbol Device:C
- removed C3, C5, C9: 10uF, Capacitor_SMD:C_0805_2012Metric_Pad1.18x1.45mm_HandSolder, symbol Device:C
- removed C8: 1uF, Capacitor_SMD:C_0805_2012Metric_Pad1.18x1.45mm_HandSolder, symbol Device:C
- removed D1: 1N5819WS, Diode_SMD:D_SOD-323, symbol Diode:1N5819WS
- removed D4: PRTR5V0U2X_215, Library:SOT143B, symbol PRTR5V0U2X_215:PRTR5V0U2X_215
- removed D5: LED, LED_SMD:LED_0603_1608Metric_Pad1.05x0.95mm_HandSolder, symbol Device:LED
- removed J1: USB_C_Receptacle_USB2.0_16P, Library:HRO_TYPE-C-31-M-12, symbol Connector:USB_C_Receptacle_USB2.0_16P
- removed J4: PinSocket_2x05_P2.00mm_Vertical, Connector_PinSocket_2.00mm:PinSocket_2x05_P2.00mm_Vertical, symbol Connector_Generic:Conn_02x05_Odd_Even
- removed J9: Conn_02x01, Connector_JST:JST_PH_B2B-PH-K_1x02_P2.00mm_Vertical, symbol Connector_Generic:Conn_02x01
- removed MK1, MK2: ICS-43434, Sensor_Audio:InvenSense_ICS-43434-6_3.5x2.65mm, symbol Sensor_Audio:ICS-43434
- removed R1, R2: 5.1K, Resistor_SMD:R_0805_2012Metric_Pad1.20x1.40mm_HandSolder, symbol Device:R
- removed R11: 10K, Resistor_SMD:R_0603_1608Metric_Pad0.98x0.95mm_HandSolder, symbol Device:R
- removed R12, R20: 1K, Resistor_SMD:R_0603_1608Metric_Pad0.98x0.95mm_HandSolder, symbol Device:R
- removed R3, R4: 100k, Resistor_SMD:R_0805_2012Metric_Pad1.20x1.40mm_HandSolder, symbol Device:R
- removed R5: 0, Jumper:SolderJumper-2_P1.3mm_Open_RoundedPad1.0x1.5mm, symbol Device:R
- removed SW1: SW_Push, Button_Switch_SMD:SW_SPST_PTS647_Sx38, symbol Switch:SW_Push
- removed U1: ESP32-S3-WROOM-1U-N8R8, PCM_Espressif:ESP32-S3-WROOM-1U, symbol RF_Module:ESP32-S3-WROOM-1
- removed U3: LT1963AEST-3.3, Package_TO_SOT_SMD:SOT-223-3_TabPin2, symbol Regulator_Linear:LT1963AxST-3.3
- added H1, H2, H3, H4: MountingHole_Pad_MP, MountingHole:MountingHole_2.2mm_M2_DIN965_Pad, symbol Mechanical:MountingHole_Pad_MP
- added J5, J7: PinHeader_2x06_P2.54mm_Vertical, Connector_PinHeader_2.54mm:PinHeader_2x06_P2.54mm_Vertical, symbol Connector_Generic:Conn_02x06_Odd_Even
- added J6, J8: BD050-10-A-0-0500-L-D, Through_hole_pin_socket:GCT_BD050-10-A-1-0500-L-D, symbol Connector_Generic:Conn_02x05_Odd_Even
Connections:
- net GND: now also H1.MP, H2.MP, H3.MP, H4.MP, J5.1 (Pin_1), J6.10 (Pin_10), J6.2 (Pin_2), J6.4 (Pin_4), J6.6 (Pin_6), J6.8 (Pin_8), J7.1 (Pin_1), J8.10 (Pin_10), J8.2 (Pin_2), J8.4 (Pin_4), J8.6 (Pin_6), J8.8 (Pin_8)
- net VCC_3V3: now also J5.11 (Pin_11), J7.2 (Pin_2), J8.1 (Pin_1)
- new net IO0: J5.9 (Pin_9), J8.3 (Pin_3)
- new net IO21: J6.3 (Pin_3), J7.9 (Pin_9)
- new net IO3: J5.7 (Pin_7), J8.5 (Pin_5)
- new net IO43: J6.1 (Pin_1), J7.11 (Pin_11)
- new net IO44: J6.5 (Pin_5), J7.7 (Pin_7)
- new net IO45: J5.5 (Pin_5), J8.7 (Pin_7)
- new net IO46: J5.3 (Pin_3), J8.9 (Pin_9)
- new net IO47: J6.7 (Pin_7), J7.5 (Pin_5)
- new net IO48: J6.9 (Pin_9), J7.3 (Pin_3)
- new net LB: J5.6 (Pin_6), J7.10 (Pin_10)
- new net SCK1: J5.10 (Pin_10), J7.6 (Pin_6)
- new net SD1: J5.8 (Pin_8), J7.8 (Pin_8)
- new net WS1: J5.12 (Pin_12), J7.4 (Pin_4)
- no-connect marks 21 -> 0
Other:
- removed sheet Eye connect
- added sheet BoardL (ESP32L.kicad_sch)
- note removed: "Board to eye adapter connector"
- note removed: "Connetions"
- note removed: "I2S"
- note removed: "I2S Mics"
- note removed: "I2S board 2"
- note removed: "SPI"
- note removed: "SPI out"
- company: (none) -> OSHE - IRL Sub-Titles
